File: PS_Test_Grid.sch (KiCad schematic (older format))
At the start: 2 parts

Commit message: Laid out HPF candidate
Parts:
- added C? (x8): C, symbol C
- added D? (x4): LED, symbol LED
- added Q? (x2): PhotoTransistor, symbol PhotoTransistor
- added R? (x24): R, symbol R
- added U? (x6): MCP6001R, symbol MCP6001R
- added U? (x2): NOA1212, symbol NOA1212
Connections:
- net labels added: GND, VDD
- wire segments 0 -> 101
Other:
- moved on the sheet: Q?, U?

Commit message: Working out the filter and amplification designs to trial
Parts:
- removed R?: R, symbol R
- added C?: C, symbol C
Connections:
- wire segments 101 -> 68
Other:
- note added: "Capacitor needs to have Z equivalent to Resistor at lowest allowed frequency.\nFor f of 1Hz, a 4.7uF cap will have 33K of Z"
- note added: "V divider resistors appear in parallel to the input\n100K = 50K\nUsing 220K and 2.2uF cuts off at .66Hz"
- moved on the sheet: R?
Changed lines of the file:
@@
 L R R?
 U 1 1 5B8B051B
-P 4650 2100
-F 0 "R?" H 4550 1950 50  0000 C CNN
-F 1 "R" H 4700 1950 50  0000 C CNN
-F 2 "" V 4580 2100 50  0001 C CNN
-F 3 "" H 4650 2100 50  0001 C CNN
-	1    4650 2100
+P 4250 2150
+F 0 "R?" H 4150 2000 50  0000 C CNN
+F 1 "R" H 4300 2000 50  0000 C CNN
+F 2 "" V 4180 2150 50  0001 C CNN
+F 3 "" H 4250 2150 50  0001 C CNN
+	1    4250 2150
 	1    0    0    -1
 $EndComp
@@
 L R R?
 U 1 1 5B8B059B
-P 4650 3150
-F 0 "R?" H 4550 3000 50  0000 C CNN
-F 1 "R" H 4700 3000 50  0000 C CNN
-F 2 "" V 4580 3150 50  0001 C CNN
-F 3 "" H 4650 3150 50  0001 C CNN
-	1    4650 3150
-	1    0    0    -1
-$EndComp
-$Comp
-L R R?
-U 1 1 5B8B0696
-P 4350 2950
-F 0 "R?" V 4250 2900 50  0000 C CNN
-F 1 "R" V 4450 2900 50  0000 C CNN
-F 2 "" V 4280 2950 50  0001 C CNN
-F 3 "" H 4350 2950 50  0001 C CNN
-	1    4350 2950
-	0    1    1    0
+P 4250 3000
+F 0 "R?" H 4150 2850 50  0000 C CNN
+F 1 "R" H 4300 2850 50  0000 C CNN
+F 2 "" V 4180 3000 50  0001 C CNN
+F 3 "" H 4250 3000 50  0001 C CNN
+	1    4250 3000
+	1    0    0    -1
 $EndComp
 $Comp
@@
 	2750 3350 2750 2800
 Wire Wire Line
-	1800 3350 2000 3350
-Wire Wire Line
-	2000 3350 2150 3350
-Wire Wire Line
-	2150 3350 2750 3350
-Wire Wire Line
-	2750 3350 3300 3350
-Wire Wire Line
-	3300 3350 3650 3350
-Wire Wire Line
-	3650 3350 4650 3350
-Wire Wire Line
-	4650 3350 5550 3350
-Wire Wire Line
-	3650 2950 3650 3350
-Wire Wire Line
-	3650 3350 3650 3650
+	1800 3350 5550 3350
+Wire Wire Line
+	3650 2950 3650 3650
 Wire Wire Line
 	5550 3350 5550 2900
@@
 	2750 1900 2750 2200
 Wire Wire Line
-	1800 1900 2100 1900
-Wire Wire Line
-	2100 1900 2300 1900
-Wire Wire Line
-	2300 1900 2750 1900
-Wire Wire Line
-	2750 1900 3550 1900
-Wire Wire Line
-	3550 1900 4650 1900
-Wire Wire Line
-	4650 1900 5550 1900
+	1800 1900 5550 1900
 Wire Wire Line
 	3550 1900 3550 1600
@@
 Connection ~ 2750 3350
 Wire Wire Line
-	3100 2500 3300 2500
-Wire Wire Line
-	3300 2500 3650 2500
-Wire Wire Line
-	3650 2500 3750 2500
+	3100 2500 3750 2500
 Wire Wire Line
 	3300 2500 3300 2650
@@
 Connection ~ 3650 2500
 Wire Wire Line
-	4650 1950 4650 1900
-Connection ~ 4650 1900
-Wire Wire Line
-	4650 2250 4650 2950
-Wire Wire Line
-	4650 2950 4650 3000
-Wire Wire Line
-	4650 3300 4650 3350
-Connection ~ 4650 3350
-Wire Wire Line
-	4500 2950 4650 2950
-Wire Wire Line
-	4650 2950 4800 2950
-Connection ~ 4650 2950
-Wire Wire Line
-	4200 2950 4150 2950
-Wire Wire Line
-	4150 2950 4150 2500
-Wire Wire Line
-	4050 2500 4150 2500
-Wire Wire Line
-	4150 2500 5350 2500
-Connection ~ 4150 2500
+	4250 2000 4250 1900
+Connection ~ 4250 1900
+Wire Wire Line
+	4250 2300 4250 2850
+Wire Wire Line
+	4250 3150 4250 3350
+Connection ~ 4250 3350
+Connection ~ 4250 2500
+Wire Wire Line
+	4050 2500 5350 2500
 Wire Wire Line
 	5950 2600 6250 2600
@@
 	5300 2700 5300 2950
 Wire Wire Line
-	5100 2950 5300 2950
-Wire Wire Line
-	5300 2950 5800 2950
+	5100 2950 5800 2950
 Connection ~ 5300 2950
 Wire Wire Line
@@
 Connection ~ 2150 3350
 Wire Wire Line
-	2150 2500 2300 2500
-Wire Wire Line
-	2300 2500 2400 2500
+	2150 2500 2400 2500
 Wire Wire Line
 	2150 2500 2150 2600
@@
 Connection ~ 2300 2500
 Wire Wire Line
-	2000 2400 2100 2400
-Wire Wire Line
-	2100 2400 2400 2400
+	2000 2400 2400 2400
 Wire Wire Line
 	2000 2400 2000 2600
@@
 	12850 1800 12850 2250
 Wire Wire Line
-	9100 1800 9750 1800
-Wire Wire Line
-	9750 1800 10850 1800
-Wire Wire Line
-	10850 1800 12050 1800
-Wire Wire Line
-	12050 1800 12850 1800
+	9100 1800 12850 1800
 Wire Wire Line
 	10850 1800 10850 1750
@@
 Connection ~ 12050 1800
 Wire Wire Line
-	12050 2300 12050 3000
-Wire Wire Line
-	12050 3000 12050 3150
+	12050 2300 12050 3150
 Wire Wire Line
 	10150 3100 10150 3550
 Wire Wire Line
-	9100 3550 10150 3550
-Wire Wire Line
-	10150 3550 10400 3550
-Wire Wire Line
-	10400 3550 10950 3550
-Wire Wire Line
-	10950 3550 12050 3550
-Wire Wire Line
-	12050 3550 12850 3550
+	9100 3550 12850 3550
 Wire Wire Line
 	10950 3550 10950 3650
@@
 Connection ~ 10400 3550
 Wire Wire Line
-	9750 2700 10150 2700
-Wire Wire Line
-	10150 2700 10400 2700
-Wire Wire Line
-	10400 2700 10750 2700
+	9750 2700 10750 2700
 Wire Wire Line
 	10400 2700 10400 2800
@@
 	11300 3000 11500 3000
 Wire Wire Line
-	11300 2500 11300 2700
-Wire Wire Line
-	11300 2700 11300 3000
+	11300 2500 11300 3000
 Connection ~ 11300 2700
 Wire Wire Line
-	11800 3000 12050 3000
-Wire Wire Line
-	12050 3000 12250 3000
+	11800 3000 12250 3000
 Connection ~ 12050 3000
 Wire Wire Line
-	12550 3000 12600 3000
-Wire Wire Line
-	12600 3000 13050 3000
+	12550 3000 13050 3000
 Wire Wire Line
 	13350 3000 13500 3000
@@
 	12600 2700 12600 3000
 Connection ~ 12600 3000
+Text Notes 3650 1850 0    60   ~ 0
+V divider resistors appear in parallel to the input\n100K = 50K\nUsing 220K and 2.2uF cuts off at .66Hz
+$Comp
+L C C?
+U 1 1 5B8B4AAD
+P 4600 3150
+F 0 "C?" H 4625 3250 50  0000 L CNN
+F 1 "C" H 4625 3050 50  0000 L CNN
+F 2 "" H 4638 3000 50  0001 C CNN
+F 3 "" H 4600 3150 50  0001 C CNN
+	1    4600 3150
+	1    0    0    -1
+$EndComp
+Wire Wire Line
+	4800 2950 4600 2950
+Wire Wire Line
+	4600 2950 4600 3000
+Wire Wire Line
+	4600 3300 4600 3350
+Connection ~ 4600 3350
+Text Notes 3700 3600 0    60   ~ 0
+Capacitor needs to have Z equivalent to Resistor at lowest allowed frequency.\nFor f of 1Hz, a 4.7uF cap will have 33K of Z
 $EndSCHEMATC

Commit message: laid out the footprints
Parts:
- removed C? (x4): C, symbol C
- removed D? (x2): LED, symbol LED
- removed Q? (x2): PhotoTransistor, symbol PhotoTransistor
- removed R? (x11): R, symbol R
- removed U? (x5): MCP6001R, symbol MCP6001R
- removed U? (x2): NOA1212, symbol NOA1212
- added C1, C11, C13, C14, C2, C4, C6, C8, C9: C, Capacitors_SMD:C_0603, symbol C
- added J1, J6: CONN_01X03, Pin_Headers:Pin_Header_Straight_1x03_Pitch2.54mm, symbol CONN_01X03
- added J10, J2, J3, J4, J5, J7, J8, J9: CONN_01X01, Pin_Headers:Pin_Header_Straight_1x01_Pitch1.00mm, symbol CONN_01X01
- added R12, R13, R14, R17, R18, R19, R20, R4: R, Capacitors_SMD:C_0603, symbol R
- added U3: MCP6001R, TO_SOT_Packages_SMD:SOT-353_SC-70-5, symbol MCP6001R
- C10, C12, C3, C5, C7: renamed from C?; footprint (none) -> Capacitors_SMD:C_0603
- D1: renamed from D?; footprint (none) -> Solutions:AM2520ZGC09_LED
- D2: renamed from D?; footprint (none) -> Solutions:VLD1235R_LED
- Q1: renamed from Q?; footprint (none) -> Solutions:EAALSTIC1708A0
- R1, R10, R11, R15, R16, R2, R3, R5, R6, R7, R8, R9: renamed from R?; footprint (none) -> Capacitors_SMD:C_0603
- U1: renamed from U?; footprint (none) -> Solutions:NOA1212CUTAG
- U2: renamed from U?; footprint (none) -> TO_SOT_Packages_SMD:SOT-353_SC-70-5
Connections:
- net labels added: GNDD, OUT_1-1, OUT_1-2, OUT_1-3, OUT_2-1, OUT_2-2, OUT_2-3, S_1, S_2, VPP
- wire segments 68 -> 109
- no-connect marks 0 -> 1
Other:
- note added: "540nm Peak Sensitivity\nNOA1212CUTAG\n"
- note added: "630nm Dominant\nVLDS1235R LED"
- note added: "630nm Peak Sensitivity"
- note added: "AM2520ZGC09\nGreen LED"
- note added: "C14 needs to have Z equivalent to R18 at lowest allowed frequency.\nFor f of 1Hz:\n0.1uF will have 1.6M\n0.68uF will have 234K\n1uF will have 159K\n3.3uF will have 48.2K\n4.7uF cap will have 33.8K\n10uF will have 15.9K"
- note added: "C7 needs to have Z equivalent to R10 at lowest allowed frequency.\nFor f of 1Hz, a 4.7uF cap will have 33K of Z"
- note added: "Still working on this with help\nhttps://www.radio-electronics.com/info/circuits/opamp_non_inverting/op_amp_non-inverting.php\nhttps://www.ieee.li/pdf/essay/single_supply_op_amp_design.pdf\n"
- note removed: "Capacitor needs to have Z equivalent to Resistor at lowest allowed frequency.\nFor f of 1Hz, a 4.7uF cap will have 33K of Z"
- moved on the sheet: C10, C12, C3, C5, C7, Q1, R1, R10, R11, R15, R16, R2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

Commit message: moved test points and cleaned schematic
Other:
- moved on the sheet: J1, J6
Changed lines of the file:
@@
 	7150 2100 7150 2400
 Wire Wire Line
-	5400 2100 10850 2100
+	5400 2100 12700 2100
 Wire Wire Line
 	7950 2100 7950 1800
@@
 Connection ~ 7950 2100
 Wire Wire Line
-	6050 2300 6050 2100
+	6050 2250 6050 2100
 Connection ~ 7150 2100
 Wire Wire Line
-	6050 2800 6050 2600
+	6050 2800 6050 2650
 Wire Wire Line
 	6050 3550 6050 3100
@@
 	7500 2700 8150 2700
 Wire Wire Line
-	7700 2700 7700 2850
+	7700 2400 7700 2850
 Wire Wire Line
 	7700 3550 7700 3150
@@
 	11250 2800 11700 2800
 Wire Wire Line
-	11550 2800 11550 3150
+	11550 2450 11550 3150
 Wire Wire Line
 	11550 3150 11300 3150
@@
 Connection ~ 7550 6850
 Wire Wire Line
-	7300 6950 7300 6850
+	7300 6550 7300 6950
 Connection ~ 7300 6850
 Wire Wire Line
@@
 Connection ~ 8000 6250
 Wire Wire Line
-	6250 6250 6250 6500
+	6250 6250 6250 6450
 Connection ~ 6900 6250
 Wire Wire Line
-	6250 6800 6250 6950
+	6250 6850 6250 6950
 Wire Wire Line
 	6250 7700 6250 7250
@@
 Connection ~ 11550 2800
 Wire Wire Line
-	12000 2800 12250 2800
+	12000 2800 13050 2800
 Wire Wire Line
 	12250 2800 12250 3000
@@
 	11000 6950 11450 6950
 Wire Wire Line
-	11300 6950 11300 7300
+	11300 6600 11300 7300
 Wire Wire Line
 	11300 7300 11050 7300
@@
 Connection ~ 11300 6950
 Wire Wire Line
-	11750 6950 12000 6950
+	11750 6950 12600 6950
 Wire Wire Line
 	12000 6950 12000 7150
@@
 Connection ~ 5850 7700
 Wire Wire Line
-	5550 6250 10600 6250
-Wire Wire Line
-	5550 7700 12000 7700
+	5550 6250 12400 6250
+Wire Wire Line
+	5550 7700 12400 7700
 Connection ~ 10600 7700
 $Comp
@@
 L CONN_01X03 J1
 U 1 1 5B92B63C
-P 12250 2250
-F 0 "J1" H 12250 2450 50  0000 C CNN
-F 1 "CONN_01X03" V 12350 2250 50  0000 C CNN
-F 2 "Pin_Headers:Pin_Header_Straight_1x03_Pitch2.54mm" H 12250 2250 50  0001 C CNN
-F 3 "" H 12250 2250 50  0001 C CNN
-	1    12250 2250
+P 13250 2900
+F 0 "J1" H 13250 3100 50  0000 C CNN
+F 1 "CONN_01X03" V 13350 2900 50  0000 C CNN
+F 2 "Pin_Headers:Pin_Header_Straight_1x03_Pitch2.54mm" H 13250 2900 50  0001 C CNN
+F 3 "" H 13250 2900 50  0001 C CNN
+	1    13250 2900
 	1    0    0    -1
 $EndComp
@@
 L CONN_01X03 J6
 U 1 1 5B92B762
-P 11950 6300
-F 0 "J6" H 11950 6500 50  0000 C CNN
-F 1 "CONN_01X03" V 12050 6300 50  0000 C CNN
-F 2 "Pin_Headers:Pin_Header_Straight_1x03_Pitch2.54mm" H 11950 6300 50  0001 C CNN
-F 3 "" H 11950 6300 50  0001 C CNN
-	1    11950 6300
-	1    0    0    -1
-$EndComp
-Text Label 11750 6200 2    60   ~ 0
-S_2
-$Comp
-L VPP #PWR05
-U 1 1 5B92BD17
-P 11450 6200
-F 0 "#PWR05" H 11450 6050 50  0001 C CNN
-F 1 "VPP" H 11450 6350 50  0000 C CNN
-F 2 "" H 11450 6200 50  0001 C CNN
-F 3 "" H 11450 6200 50  0001 C CNN
-	1    11450 6200
-	1    0    0    -1
-$EndComp
-$Comp
-L GNDD #PWR06
-U 1 1 5B92BE1E
-P 11450 6500
-F 0 "#PWR06" H 11450 6250 50  0001 C CNN
-F 1 "GNDD" H 11450 6350 50  0000 C CNN
-F 2 "" H 11450 6500 50  0001 C CNN
-F 3 "" H 11450 6500 50  0001 C CNN
-	1    11450 6500
-	1    0    0    -1
-$EndComp
-Wire Wire Line
-	11750 6400 11450 6400
-Wire Wire Line
-	11450 6400 11450 6500
-Wire Wire Line
-	11750 6300 11450 6300
-Wire Wire Line
-	11450 6300 11450 6200
-Text Label 12050 2150 2    60   ~ 0
-S_1
-$Comp
-L GND #PWR07
-U 1 1 5B92C258
-P 11700 2450
-F 0 "#PWR07" H 11700 2200 50  0001 C CNN
-F 1 "GND" H 11700 2300 50  0000 C CNN
-F 2 "" H 11700 2450 50  0001 C CNN
-F 3 "" H 11700 2450 50  0001 C CNN
-	1    11700 2450
-	1    0    0    -1
-$EndComp
-$Comp
-L VDD #PWR08
-U 1 1 5B92C2E1
-P 11700 2100
-F 0 "#PWR08" H 11700 1950 50  0001 C CNN
-F 1 "VDD" H 11700 2250 50  0000 C CNN
-F 2 "" H 11700 2100 50  0001 C CNN
-F 3 "" H 11700 2100 50  0001 C CNN
-	1    11700 2100
-	1    0    0    -1
-$EndComp
-Wire Wire Line
-	12050 2250 11700 2250
-Wire Wire Line
-	11700 2250 11700 2100
-Wire Wire Line
-	12050 2350 11700 2350
-Wire Wire Line
-	11700 2350 11700 2450
+P 12800 7050
+F 0 "J6" H 12800 7250 50  0000 C CNN
+F 1 "CONN_01X03" V 12900 7050 50  0000 C CNN
+F 2 "Pin_Headers:Pin_Header_Straight_1x03_Pitch2.54mm" H 12800 7050 50  0001 C CNN
+F 3 "" H 12800 7050 50  0001 C CNN
+	1    12800 7050
+	1    0    0    -1
+$EndComp
+Wire Wire Line
+	12600 7150 12400 7150
+Wire Wire Line
+	12400 7150 12400 7700
+Wire Wire Line
+	12400 7050 12600 7050
+Wire Wire Line
+	12400 6250 12400 7050
+Wire Wire Line
+	13050 2900 12700 2900
+Wire Wire Line
+	13050 3000 12700 3000
+Wire Wire Line
+	12700 3550 12700 3000
 $Comp
 L CONN_01X01 J2
@@
 	-1   0    0    1
 $EndComp
-Text Label 7850 2700 1    60   ~ 0
+Text Label 7700 2400 0    60   ~ 0
 OUT_1-1
-Text Label 8650 2700 1    60   ~ 0
+Text Label 9900 2350 0    60   ~ 0
 OUT_1-2
-Text Label 10450 2700 1    60   ~ 0
+Text Label 11550 2450 0    60   ~ 0
 OUT_1-3
 Text Label 4650 2800 0    60   ~ 0
@@
 OUT_1-1
 $Comp
-L GND #PWR09
+L GND #PWR05
 U 1 1 5B92D807
 P 4750 3100
-F 0 "#PWR09" H 4750 2850 50  0001 C CNN
+F 0 "#PWR05" H 4750 2850 50  0001 C CNN
 F 1 "GND" H 4750 2950 50  0000 C CNN
 F 2 "" H 4750 3100 50  0001 C CNN
@@
 Wire Wire Line
 	4750 3000 4750 3100
-Text Label 7450 6850 1    60   ~ 0
+Text Label 7300 6550 0    60   ~ 0
 OUT_2-1
-Text Label 8350 6850 1    60   ~ 0
+Text Label 9600 6550 0    60   ~ 0
 OUT_2-2
-Text Label 10150 6850 1    60   ~ 0
+Text Label 11300 6600 0    60   ~ 0
 OUT_2-3
 $Comp
@@
 OUT_2-3
 $Comp
-L GNDD #PWR010
+L GNDD #PWR06
 U 1 1 5B92E777
 P 5000 7400
-F 0 "#PWR010" H 5000 7150 50  0001 C CNN
+F 0 "#PWR06" H 5000 7150 50  0001 C CNN
 F 1 "GNDD" H 5000 7250 50  0000 C CNN
 F 2 "" H 5000 7400 50  0001 C CNN
@@
 Wire Wire Line
 	5000 7200 5000 7400
-Text Label 12000 6950 0    60   ~ 0
+Text Label 12100 6950 0    60   ~ 0
 S_2
-Text Label 12250 2800 0    60   ~ 0
+Text Label 12350 2800 0    60   ~ 0
 S_1
 Text Notes 6550 6000 0    60   ~ 0
@@
 AM2520ZGC09\nGreen LED
 Wire Wire Line
-	5400 3550 12250 3550
+	5400 3550 12700 3550
 Wire Wire Line
 	10650 2700 9900 2700
@@
 	9600 7150 9400 7150
 Connection ~ 9600 6850
+Wire Wire Line
+	12700 2900 12700 2100
+Connection ~ 10850 2100
+Connection ~ 12250 2800
+Connection ~ 12250 3550
+Connection ~ 10600 6250
+Connection ~ 12000 7700
+Connection ~ 12000 6950
 $EndSCHEMATC
