File: PS_Test_Grid.sch (KiCad schematic (older format))
At the start: 50 parts, among them J1 CONN_01X03, J10 CONN_01X01, J2 CONN_01X01, J3 CONN_01X01, J4 CONN_01X01, J5 CONN_01X01, J6 CONN_01X03, J7 CONN_01X01, J8 CONN_01X01, J9 CONN_01X01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

Commit message: working out component value scheme
Parts:
- D1, D2: symbol LED -> LED-RESCUE-PS_Test_Grid
- R11: value R -> 330K
- R13, R14, R17: value R -> 100K
- R3, R4, R9: value R -> 220K
- U2, U3: symbol MCP6001R -> MCP6001R-RESCUE-PS_Test_Grid
Other:
- note added: "BW1 = 1/2PI(R3/2)C6 = \nBW2 = 1/2PI*R4*C3 = \nBW3 = 1/2PI*R10*C7 =\n\nBW1 = 0.1*BW2 | 0.1*BW3"
- note added: "BW1 AT C13\n0.1uF = 31.83Hz\n1uF = 3.18Hz\n2.2uF = 1.44Hz\n3.3uF = 0.96Hz\n4.7uF = 0.68Hz"
- note added: "BW1 for C6\n0.1uF = 14.47Hz\n1uF = 1.45Hz\n2.2uF = 0.66Hz\n3.3uF = 0.44Hz\n4.7uF = 0.31Hz"
- note added: "BW2 AT C3\n0.022uF = 72Hz\n0.033uF = 48Hz\n0.047uF = 34Hz\n0.1uF = 16.9Hz\n1uF = 1.59Hz\n2.2uF = 0.72Hz\n3.3uF = 0.48Hz\n4.7uF = 0.34Hz"
- note added: "BW2 for C3\n0.022uF = 32.88Hz\n0.033uF = 21.92Hz\n0.047uF = 15.39Hz\n0.1uF = 7.23Hz\n1uF = 0.72Hz\n2.2uF = 0.33Hz\n3.3uF = 0.22Hz\n4.7uF = 0.15Hz"
- note added: "BW3 = BW2"
- note added: "C14 needs to have Z equivalent to R18 at lowest allowed frequency.\n\nFor f of 1Hz:\n0.1uF will have 1.6M\n0.68uF will have 234K\n1uF will have 159K\n3.3uF will have 48.2K\n4.7uF cap will have 33.8K\n10uF will have 15.9K"
- note added: "C7 Z AT 14.5Hz (BW1*10 @ 1uF)\n0.1uF = 110K\n1uF = 11K\n2.2uF = 5K\n3.3uF = 3.3K\n4.7uF = 2.3K"
- note added: "C7 Z AT 6.6Hz (BW1*10 at 2.2uF)\n0.1uF = 241K\n1uF = 24K\n2.2uF = 11K\n3.3uF = 7.3K\n4.7uF = 5K"
- note added: "C7 needs to have Z equivalent to R10 at lowest allowed frequency.\nR11 should equal R4+(R3/2) to reduce input bias current erros.\nChoose bypass C6 to set CMR dropoff"
- note added: "For f of 0.8Hz:\n0.1uF will have \n0.68uF will have \n1uF will have \n3.3uF will have \n4.7uF cap will have \n10uF will have"
- note added: "G = 1+R11/R10\n"
- note added: "Still working on this with help\nhttps://www.radio-electronics.com/info/circuits/opamp_non_inverting/op_amp_non-inverting.php\nhttps://www.ieee.li/pdf/essay/single_supply_op_amp_design.pdf\nhttps://www.analog.com/en/analog-dialogue/articles/avoiding-op-amp-instability-problems.html"
- note added: "V divider resistors appear in parallel to the input\n220K = 110K\nUsing 220K and 2.2uF cuts off at .66Hz"
- note added: "V divider resistors appear in parallel to the input\nX = R3/2"
- note added: "Z = 1/2PI*f*C"
- note removed: "C14 needs to have Z equivalent to R18 at lowest allowed frequency.\nFor f of 1Hz:\n0.1uF will have 1.6M\n0.68uF will have 234K\n1uF will have 159K\n3.3uF will have 48.2K\n4.7uF cap will have 33.8K\n10uF will have 15.9K"
- note removed: "C7 needs to have Z equivalent to R10 at lowest allowed frequency.\nFor f of 1Hz, a 4.7uF cap will have 33K of Z"
- note removed: "Still working on this with help\nhttps://www.radio-electronics.com/info/circuits/opamp_non_inverting/op_amp_non-inverting.php\nhttps://www.ieee.li/pdf/essay/single_supply_op_amp_design.pdf\n"
- note removed: "V divider resistors appear in parallel to the input\n100K = 50K\nUsing 220K and 2.2uF cuts off at .66Hz"
Changed lines of the file:
@@
 EESchema Schematic File Version 2
+LIBS:PS_Test_Grid-rescue
 LIBS:power
 LIBS:device
@@
 $EndComp
 $Comp
-L MCP6001R U2
+L MCP6001R-RESCUE-PS_Test_Grid U2
 U 1 1 5B8AF47D
 P 10950 2800
@@
 $EndComp
 $Comp
-L LED D2
+L LED-RESCUE-PS_Test_Grid D2
 U 1 1 5B8AFAB0
 P 6250 6650
@@
 $EndComp
 $Comp
-L LED D1
+L LED-RESCUE-PS_Test_Grid D1
 U 1 1 5B8AFC0D
 P 6050 2450
@@
 P 11150 3150
 F 0 "R11" V 11050 3100 50  0000 C CNN
-F 1 "R" V 11250 3100 50  0000 C CNN
+F 1 "330K" V 11250 3100 50  0000 C CNN
 F 2 "Capacitors_SMD:C_0603" V 11080 3150 50  0001 C CNN
 F 3 "" H 11150 3150 50  0001 C CNN
@@
 U 1 1 5B8B051B
 P 9150 2600
-F 0 "R3" H 9050 2450 50  0000 C CNN
-F 1 "R" H 9200 2450 50  0000 C CNN
+F 0 "R3" H 9050 2600 50  0000 C CNN
+F 1 "220K" H 9300 2600 50  0000 C CNN
 F 2 "Capacitors_SMD:C_0603" V 9080 2600 50  0001 C CNN
 F 3 "" H 9150 2600 50  0001 C CNN
@@
 U 1 1 5B8B059B
 P 9150 3200
-F 0 "R9" H 9050 3050 50  0000 C CNN
-F 1 "R" H 9200 3050 50  0000 C CNN
+F 0 "R9" H 9050 3200 50  0000 C CNN
+F 1 "220K" H 9300 3200 50  0000 C CNN
 F 2 "Capacitors_SMD:C_0603" V 9080 3200 50  0001 C CNN
 F 3 "" H 9150 3200 50  0001 C CNN
@@
 Connection ~ 7300 7700
 Text Notes 8050 2050 0    60   ~ 0
-V divider resistors appear in parallel to the input\n100K = 50K\nUsing 220K and 2.2uF cuts off at .66Hz
+V divider resistors appear in parallel to the input\nX = R3/2
 $Comp
 L C C7
@@
 	10050 3550 10050 3500
 Connection ~ 10050 3550
-Text Notes 8600 3800 0    60   ~ 0
-C7 needs to have Z equivalent to R10 at lowest allowed frequency.\nFor f of 1Hz, a 4.7uF cap will have 33K of Z
-Text Notes 5900 4450 0    60   ~ 0
-Still working on this with help\nhttps://www.radio-electronics.com/info/circuits/opamp_non_inverting/op_amp_non-inverting.php\nhttps://www.ieee.li/pdf/essay/single_supply_op_amp_design.pdf\n
+Text Notes 13050 4350 0    60   ~ 0
+C7 needs to have Z equivalent to R10 at lowest allowed frequency.\nR11 should equal R4+(R3/2) to reduce input bias current erros.\nChoose bypass C6 to set CMR dropoff
+Text Notes 750  9650 0    60   ~ 0
+Still working on this with help\nhttps://www.radio-electronics.com/info/circuits/opamp_non_inverting/op_amp_non-inverting.php\nhttps://www.ieee.li/pdf/essay/single_supply_op_amp_design.pdf\nhttps://www.analog.com/en/analog-dialogue/articles/avoiding-op-amp-instability-problems.html
 NoConn ~ 6800 2850
 $Comp
@@
 P 9500 2900
 F 0 "R4" V 9400 2850 50  0000 C CNN
-F 1 "R" V 9600 2850 50  0000 C CNN
+F 1 "220K" V 9600 2900 50  0000 C CNN
 F 2 "Capacitors_SMD:C_0603" V 9430 2900 50  0001 C CNN
 F 3 "" H 9500 2900 50  0001 C CNN
@@
 	5550 6850 5550 7700
 $Comp
-L MCP6001R U3
+L MCP6001R-RESCUE-PS_Test_Grid U3
 U 1 1 5B91F924
 P 10700 6950
@@
 U 1 1 5B91F936
 P 8900 6850
-F 0 "R13" H 8800 6700 50  0000 C CNN
-F 1 "R" H 8950 6700 50  0000 C CNN
+F 0 "R13" H 8750 6850 50  0000 C CNN
+F 1 "100K" H 9050 6850 50  0000 C CNN
 F 2 "Capacitors_SMD:C_0603" V 8830 6850 50  0001 C CNN
 F 3 "" H 8900 6850 50  0001 C CNN
@@
 U 1 1 5B91F93C
 P 8900 7400
-F 0 "R17" H 8800 7250 50  0000 C CNN
-F 1 "R" H 8950 7250 50  0000 C CNN
+F 0 "R17" H 9050 7450 50  0000 C CNN
+F 1 "100K" H 9050 7350 50  0000 C CNN
 F 2 "Capacitors_SMD:C_0603" V 8830 7400 50  0001 C CNN
 F 3 "" H 8900 7400 50  0001 C CNN
@@
 Connection ~ 10350 7300
 Text Notes 8400 6200 0    60   ~ 0
-V divider resistors appear in parallel to the input\n100K = 50K\nUsing 220K and 2.2uF cuts off at .66Hz
+V divider resistors appear in parallel to the input\n220K = 110K\nUsing 220K and 2.2uF cuts off at .66Hz
 $Comp
 L C C14
@@
 	9800 7700 9800 7650
 Connection ~ 9800 7700
-Text Notes 9600 8600 0    60   ~ 0
-C14 needs to have Z equivalent to R18 at lowest allowed frequency.\nFor f of 1Hz:\n0.1uF will have 1.6M\n0.68uF will have 234K\n1uF will have 159K\n3.3uF will have 48.2K\n4.7uF cap will have 33.8K\n10uF will have 15.9K
+Text Notes 9600 8650 0    60   ~ 0
+C14 needs to have Z equivalent to R18 at lowest allowed frequency.\n\nFor f of 1Hz:\n0.1uF will have 1.6M\n0.68uF will have 234K\n1uF will have 159K\n3.3uF will have 48.2K\n4.7uF cap will have 33.8K\n10uF will have 15.9K
 $Comp
 L R R14
@@
 P 9250 7150
 F 0 "R14" V 9150 7100 50  0000 C CNN
-F 1 "R" V 9350 7100 50  0000 C CNN
+F 1 "100K" V 9350 7150 50  0000 C CNN
 F 2 "Capacitors_SMD:C_0603" V 9180 7150 50  0001 C CNN
 F 3 "" H 9250 7150 50  0001 C CNN
@@
 	13050 3000 12700 3000
 Wire Wire Line
-	12700 3550 12700 3000
+	12700 3000 12700 3550
 $Comp
 L CONN_01X01 J2
@@
 AM2520ZGC09\nGreen LED
 Wire Wire Line
-	5400 3550 12700 3550
+	12700 3550 5400 3550
 Wire Wire Line
 	10650 2700 9900 2700
@@
 Connection ~ 12000 7700
 Connection ~ 12000 6950
+Text Notes 11200 8650 0    60   ~ 0
+For f of 0.8Hz:\n0.1uF will have \n0.68uF will have \n1uF will have \n3.3uF will have \n4.7uF cap will have \n10uF will have
+Text Notes 9600 8850 0    60   ~ 0
+Z = 1/2PI*f*C
+Text Notes 5450 4200 0    60   ~ 0
+BW1 = 1/2PI(R3/2)C6 = \nBW2 = 1/2PI*R4*C3 = \nBW3 = 1/2PI*R10*C7 =\n\nBW1 = 0.1*BW2  |  0.1*BW3
+Text Notes 1550 2700 0    60   ~ 0
+BW1 for C6\n0.1uF = 14.47Hz\n1uF = 1.45Hz\n2.2uF = 0.66Hz\n3.3uF = 0.44Hz\n4.7uF = 0.31Hz
+Text Notes 1400 7150 0    60   ~ 0
+BW1 AT C13\n0.1uF = 31.83Hz\n1uF = 3.18Hz\n2.2uF = 1.44Hz\n3.3uF = 0.96Hz\n4.7uF = 0.68Hz
+Text Notes 1550 4200 0    60   ~ 0
+BW2 for C3\n0.022uF = 32.88Hz\n0.033uF = 21.92Hz\n0.047uF = 15.39Hz\n0.1uF = 7.23Hz\n1uF = 0.72Hz\n2.2uF = 0.33Hz\n3.3uF = 0.22Hz\n4.7uF = 0.15Hz
+Text Notes 1550 4700 0    60   ~ 0
+BW3 = BW2
+Text Notes 8600 4250 0    60   ~ 0
+C7 Z AT 6.6Hz (BW1*10 at 2.2uF)\n0.1uF = 241K\n1uF = 24K\n2.2uF = 11K\n3.3uF = 7.3K\n4.7uF = 5K
+Text Notes 1400 8300 0    60   ~ 0
+BW2 AT C3\n0.022uF = 72Hz\n0.033uF = 48Hz\n0.047uF = 34Hz\n0.1uF = 16.9Hz\n1uF = 1.59Hz\n2.2uF = 0.72Hz\n3.3uF = 0.48Hz\n4.7uF = 0.34Hz
+Text Notes 10550 4250 0    60   ~ 0
+C7 Z AT 14.5Hz (BW1*10 @ 1uF)\n0.1uF = 110K\n1uF = 11K\n2.2uF = 5K\n3.3uF = 3.3K\n4.7uF = 2.3K
+Text Notes 9550 4450 0    60   ~ 0
+Z = 1/2PI*f*C
+Text Notes 13900 3400 0    60   ~ 0
+G = 1+R11/R10\n
 $EndSCHEMATC

Commit message: saved notes
Other:
- moved on the sheet: J1
Changed lines of the file:
@@
 	7150 3550 7150 3000
 Wire Wire Line
-	8050 3150 8050 3850
+	8050 3150 8050 3550
+Wire Wire Line
+	8050 3550 8050 3850
 Wire Wire Line
 	10850 3550 10850 3100
@@
 	7150 2100 7150 2400
 Wire Wire Line
-	5400 2100 12700 2100
+	5400 2100 5700 2100
+Wire Wire Line
+	5700 2100 6050 2100
+Wire Wire Line
+	6050 2100 6400 2100
+Wire Wire Line
+	6400 2100 6700 2100
+Wire Wire Line
+	6700 2100 7150 2100
+Wire Wire Line
+	7150 2100 7950 2100
+Wire Wire Line
+	7950 2100 9150 2100
+Wire Wire Line
+	9150 2100 10850 2100
+Wire Wire Line
+	10850 2100 12700 2100
 Wire Wire Line
 	7950 2100 7950 1800
@@
 Connection ~ 7150 3550
 Wire Wire Line
-	7500 2700 8150 2700
-Wire Wire Line
-	7700 2400 7700 2850
+	7500 2700 7700 2700
+Wire Wire Line
+	7700 2700 8050 2700
+Wire Wire Line
+	8050 2700 8150 2700
+Wire Wire Line
+	7700 2400 7700 2700
+Wire Wire Line
+	7700 2700 7700 2850
 Wire Wire Line
 	7700 3550 7700 3150
@@
 Connection ~ 9150 2100
 Wire Wire Line
-	9150 2750 9150 3050
+	9150 2750 9150 2900
+Wire Wire Line
+	9150 2900 9150 3050
 Wire Wire Line
 	9150 3550 9150 3350
@@
 Connection ~ 9150 2900
 Wire Wire Line
-	11250 2800 11700 2800
-Wire Wire Line
-	11550 2450 11550 3150
+	11250 2800 11550 2800
+Wire Wire Line
+	11550 2800 11700 2800
+Wire Wire Line
+	11550 2450 11550 2800
+Wire Wire Line
+	11550 2800 11550 3150
 Wire Wire Line
 	11550 3150 11300 3150
@@
 	10600 2900 10600 3150
 Wire Wire Line
-	10500 3150 11000 3150
+	10500 3150 10600 3150
+Wire Wire Line
+	10600 3150 11000 3150
 Connection ~ 10600 3150
 Wire Wire Line
@@
 Connection ~ 6550 3550
 Wire Wire Line
-	6550 2700 6800 2700
+	6550 2700 6700 2700
+Wire Wire Line
+	6700 2700 6800 2700
 Wire Wire Line
 	6550 2700 6550 2800
@@
 Connection ~ 6700 2700
 Wire Wire Line
-	6300 2600 6800 2600
+	6300 2600 6400 2600
+Wire Wire Line
+	6400 2600 6800 2600
 Wire Wire Line
 	6300 2600 6300 2800
@@
 Connection ~ 7550 7700
 Wire Wire Line
-	6900 6850 7900 6850
+	6900 6850 7300 6850
+Wire Wire Line
+	7300 6850 7550 6850
+Wire Wire Line
+	7550 6850 7900 6850
 Wire Wire Line
 	7550 6850 7550 6950
@@
 Connection ~ 7550 6850
 Wire Wire Line
-	7300 6550 7300 6950
+	7300 6550 7300 6850
+Wire Wire Line
+	7300 6850 7300 6950
 Connection ~ 7300 6850
 Wire Wire Line
@@
 Connection ~ 11550 2800
 Wire Wire Line
-	12000 2800 13050 2800
+	12000 2800 12250 2800
+Wire Wire Line
+	12250 2800 12800 2800
 Wire Wire Line
 	12250 2800 12250 3000
@@
 Connection ~ 8900 6250
 Wire Wire Line
-	8900 7000 8900 7250
+	8900 7000 8900 7150
+Wire Wire Line
+	8900 7150 8900 7250
 Wire Wire Line
 	8900 7700 8900 7550
@@
 Connection ~ 8900 7150
 Wire Wire Line
-	11000 6950 11450 6950
-Wire Wire Line
-	11300 6600 11300 7300
+	11000 6950 11300 6950
+Wire Wire Line
+	11300 6950 11450 6950
+Wire Wire Line
+	11300 6600 11300 6950
+Wire Wire Line
+	11300 6950 11300 7300
 Wire Wire Line
 	11300 7300 11050 7300
@@
 	10350 7050 10350 7300
 Wire Wire Line
-	10250 7300 10750 7300
+	10250 7300 10350 7300
+Wire Wire Line
+	10350 7300 10750 7300
 Connection ~ 10350 7300
 Text Notes 8400 6200 0    60   ~ 0
@@
 Connection ~ 11300 6950
 Wire Wire Line
-	11750 6950 12600 6950
+	11750 6950 12000 6950
+Wire Wire Line
+	12000 6950 12600 6950
 Wire Wire Line
 	12000 6950 12000 7150
@@
 Connection ~ 5850 7700
 Wire Wire Line
-	5550 6250 12400 6250
-Wire Wire Line
-	5550 7700 12400 7700
+	5550 6250 5850 6250
+Wire Wire Line
+	5850 6250 6250 6250
+Wire Wire Line
+	6250 6250 6900 6250
+Wire Wire Line
+	6900 6250 8000 6250
+Wire Wire Line
+	8000 6250 8900 6250
+Wire Wire Line
+	8900 6250 10600 6250
+Wire Wire Line
+	10600 6250 12400 6250
+Wire Wire Line
+	5550 7700 5850 7700
+Wire Wire Line
+	5850 7700 6250 7700
+Wire Wire Line
+	6250 7700 7300 7700
+Wire Wire Line
+	7300 7700 7550 7700
+Wire Wire Line
+	7550 7700 8100 7700
+Wire Wire Line
+	8100 7700 8550 7700
+Wire Wire Line
+	8550 7700 8900 7700
+Wire Wire Line
+	8900 7700 9800 7700
+Wire Wire Line
+	9800 7700 10600 7700
+Wire Wire Line
+	10600 7700 12000 7700
+Wire Wire Line
+	12000 7700 12400 7700
 Connection ~ 10600 7700
 $Comp
@@
 L CONN_01X03 J1
 U 1 1 5B92B63C
-P 13250 2900
-F 0 "J1" H 13250 3100 50  0000 C CNN
-F 1 "CONN_01X03" V 13350 2900 50  0000 C CNN
-F 2 "Pin_Headers:Pin_Header_Straight_1x03_Pitch2.54mm" H 13250 2900 50  0001 C CNN
-F 3 "" H 13250 2900 50  0001 C CNN
-	1    13250 2900
+P 13000 2900
+F 0 "J1" H 13000 3100 50  0000 C CNN
+F 1 "CONN_01X03" V 13100 2900 50  0000 C CNN
+F 2 "Pin_Headers:Pin_Header_Straight_1x03_Pitch2.54mm" H 13000 2900 50  0001 C CNN
+F 3 "" H 13000 2900 50  0001 C CNN
+	1    13000 2900
 	1    0    0    -1
 $EndComp
@@
 	12400 6250 12400 7050
 Wire Wire Line
-	13050 2900 12700 2900
-Wire Wire Line
-	13050 3000 12700 3000
+	12800 2900 12700 2900
+Wire Wire Line
+	12800 3000 12700 3000
 Wire Wire Line
 	12700 3000 12700 3550
@@
 AM2520ZGC09\nGreen LED
 Wire Wire Line
-	12700 3550 5400 3550
+	12700 3550 12250 3550
+Wire Wire Line
+	12250 3550 10850 3550
+Wire Wire Line
+	10850 3550 10050 3550
+Wire Wire Line
+	10050 3550 9150 3550
+Wire Wire Line
+	9150 3550 8750 3550
+Wire Wire Line
+	8750 3550 8050 3550
+Wire Wire Line
+	8050 3550 7700 3550
+Wire Wire Line
+	7700 3550 7150 3550
+Wire Wire Line
+	7150 3550 6550 3550
+Wire Wire Line
+	6550 3550 6300 3550
+Wire Wire Line
+	6300 3550 6050 3550
+Wire Wire Line
+	6050 3550 5700 3550
+Wire Wire Line
+	5700 3550 5400 3550
 Wire Wire Line
 	10650 2700 9900 2700
 Wire Wire Line
-	9900 2350 9900 2900
+	9900 2350 9900 2700
+Wire Wire Line
+	9900 2700 9900 2900
 Wire Wire Line
 	9900 2900 9650 2900
 Wire Wire Line
-	8750 2900 9350 2900
+	8750 2900 9150 2900
+Wire Wire Line
+	9150 2900 9350 2900
 Wire Wire Line
 	8750 3050 8750 2900
@@
 	8550 6550 9600 6550
 Wire Wire Line
-	9600 6550 9600 7150
+	9600 6550 9600 6850
+Wire Wire Line
+	9600 6850 9600 7150
 Wire Wire Line
 	9600 6850 10400 6850
 Wire Wire Line
-	8550 7150 9100 7150
+	8550 7150 8900 7150
+Wire Wire Line
+	8900 7150 9100 7150
 Wire Wire Line
 	8550 7250 8550 7150

Commit message: upgraded to KiCad 5
Parts:
- C1, C10, C11, C12, C13, C14, C2, C3, C4, C5, C6, C7, C8, C9: symbol C -> Device:C
- D1, D2: symbol LED-RESCUE-PS_Test_Grid -> PS_Test_Grid-rescue:LED-RESCUE-PS_Test_Grid
- J1, J6: symbol CONN_01X03 -> PS_Test_Grid-rescue:CONN_01X03
- J10, J2, J3, J4, J5, J7, J8, J9: symbol CONN_01X01 -> PS_Test_Grid-rescue:CONN_01X01
- Q1: symbol PhotoTransistor -> Solutions:PhotoTransistor
- R1, R2, R6, R7: footprint Capacitors_SMD:C_0603 -> Capacitors_SMD:C_0402; symbol R -> Device:R
- R10, R11, R12, R13, R14, R15, R16, R17, R18, R19, R20, R3, R4, R5, R8, R9: symbol R -> Device:R
- U1: symbol NOA1212 -> Solutions:NOA1212
- U2, U3: symbol MCP6001R-RESCUE-PS_Test_Grid -> PS_Test_Grid-rescue:MCP6001R-RESCUE-PS_Test_Grid
