File: PS_Test_Grid.sch (KiCad schematic (older format))
At the start: 52 parts, among them J1 CONN_01X03, J10 CONN_01X01, J2 CONN_01X01, J3 CONN_01X01, J4 CONN_01X01, J5 CONN_01X01, J6 CONN_01X03, J7 CONN_01X01, J8 CONN_01X01, J9 CONN_01X01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

Commit message: adjusted protection diode. Reroute
Parts:
- removed C2, C9: C, Capacitors_SMD:C_0603, symbol Device:C
- D3, D4: footprint Solutions:NSR20F30NXT5G_DIODE -> Solutions:RB751S40T5G_DIODE
Connections:
- net GND: no longer D3.2 (A)
- net GNDD: no longer D4.2 (A)
- net VDD: now also D3.2 (A); no longer C1.1, D3.1 (K), R1.1, R2.1, U1.1 (Vdd), U2.2 (V+)
- net VPP: now also D4.2 (A); no longer C8.1, D4.1 (K), Q1.1 (C), U3.2 (V+)
- new net DVDD: C1.1, D3.1 (K), R1.1, R2.1, U1.1 (Vdd), U2.2 (V+)
- new net DVPP: C8.1, D4.1 (K), Q1.1 (C), U3.2 (V+)
Other:
- note added: "RB751S40T5G"
- note removed: "NSR20F30NXT5G"
- moved on the sheet: C1, C8, D3, D4
Changed lines of the file:
@@
 P 6800 6550
 F 0 "Q1" H 7000 6700 60  0000 C CNN
-F 1 "PhotoTransistor" H 6900 6950 60  0000 C CNN
+F 1 "PhotoTransistor" H 6850 6150 60  0000 C CNN
 F 2 "Solutions:EAALSTIC1708A0" H 6800 6550 60  0001 C CNN
 F 3 "" H 6800 6550 60  0000 C CNN
@@
 	1    0    0    -1
 $EndComp
-Text Notes 6550 6100 0    60   ~ 0
+Text Notes 6500 5900 0    60   ~ 0
 EAALSTIC1708A0\n
 $Comp
@@
 L power:VDD #PWR01
 U 1 1 5B8AF6E2
-P 7950 1800
-F 0 "#PWR01" H 7950 1650 50  0001 C CNN
-F 1 "VDD" H 7950 1950 50  0000 C CNN
-F 2 "" H 7950 1800 50  0001 C CNN
-F 3 "" H 7950 1800 50  0001 C CNN
-	1    7950 1800
+P 7950 1650
+F 0 "#PWR01" H 7950 1500 50  0001 C CNN
+F 1 "VDD" H 7950 1800 50  0000 C CNN
+F 2 "" H 7950 1650 50  0001 C CNN
+F 3 "" H 7950 1650 50  0001 C CNN
+	1    7950 1650
 	1    0    0    -1
 $EndComp
@@
 Connection ~ 8050 3550
 Wire Wire Line
-	5400 2100 5700 2100
-Wire Wire Line
-	7950 2100 7950 1800
-Connection ~ 7950 2100
-Wire Wire Line
-	6050 2250 6050 2100
+	7950 1850 7950 1650
+Connection ~ 7950 1850
+Wire Wire Line
+	6050 2250 6050 1850
 Wire Wire Line
 	6050 2800 6050 2650
@@
 Connection ~ 8050 2700
 Wire Wire Line
-	9150 2450 9150 2100
-Connection ~ 9150 2100
+	9150 2450 9150 1850
+Connection ~ 9150 1850
 Wire Wire Line
 	9150 2750 9150 2900
@@
 Connection ~ 6400 2600
 Wire Wire Line
-	8000 6250 8000 5900
+	8000 6000 8000 5900
 Wire Wire Line
 	7300 7700 7300 7250
@@
 Connection ~ 7300 6850
 Wire Wire Line
-	6900 6250 6900 6350
-Wire Wire Line
 	6250 6850 6250 6950
 Wire Wire Line
 	6250 7700 6250 7250
 Connection ~ 7300 7700
-Text Notes 8050 2050 0    60   ~ 0
+Text Notes 8100 1750 0    60   ~ 0
 V divider resistors appear in parallel to the input\nX = R3/2
 $Comp
@@
 $EndComp
 $Comp
-L Device:C C2
-U 1 1 5B91CB99
-P 5700 2650
-F 0 "C2" H 5725 2750 50  0000 L CNN
-F 1 "C" H 5725 2550 50  0000 L CNN
-F 2 "Capacitors_SMD:C_0603" H 5738 2500 50  0001 C CNN
-F 3 "" H 5700 2650 50  0001 C CNN
-	1    5700 2650
-	1    0    0    -1
-$EndComp
-$Comp
 L Device:C C1
 U 1 1 5B91CC4A
-P 5400 2650
-F 0 "C1" H 5425 2750 50  0000 L CNN
-F 1 "C" H 5425 2550 50  0000 L CNN
-F 2 "Capacitors_SMD:C_0603" H 5438 2500 50  0001 C CNN
-F 3 "" H 5400 2650 50  0001 C CNN
-	1    5400 2650
-	1    0    0    -1
-$EndComp
-Wire Wire Line
-	5700 2500 5700 2100
-Wire Wire Line
-	5700 2800 5700 3550
+P 5600 2650
+F 0 "C1" H 5625 2750 50  0000 L CNN
+F 1 "C" H 5625 2550 50  0000 L CNN
+F 2 "Capacitors_SMD:C_0603" H 5638 2500 50  0001 C CNN
+F 3 "" H 5600 2650 50  0001 C CNN
+	1    5600 2650
+	1    0    0    -1
+$EndComp
 Connection ~ 6050 3550
 Wire Wire Line
-	5400 2500 5400 2100
-Wire Wire Line
-	5400 2800 5400 3550
-Connection ~ 5700 3550
+	5600 2800 5600 3550
 $Comp
 L Device:C C4
@@
 $EndComp
 $Comp
-L Device:C C9
-U 1 1 5B91E34E
+L Device:C C8
+U 1 1 5B91E354
 P 5850 6700
-F 0 "C9" H 5875 6800 50  0000 L CNN
+F 0 "C8" H 5875 6800 50  0000 L CNN
 F 1 "C" H 5875 6600 50  0000 L CNN
 F 2 "Capacitors_SMD:C_0603" H 5888 6550 50  0001 C CNN
@@
 	1    0    0    -1
 $EndComp
-$Comp
-L Device:C C8
-U 1 1 5B91E354
-P 5550 6700
-F 0 "C8" H 5575 6800 50  0000 L CNN
-F 1 "C" H 5575 6600 50  0000 L CNN
-F 2 "Capacitors_SMD:C_0603" H 5588 6550 50  0001 C CNN
-F 3 "" H 5550 6700 50  0001 C CNN
-	1    5550 6700
-	1    0    0    -1
-$EndComp
-Wire Wire Line
-	5850 6250 5850 6550
-Wire Wire Line
-	5550 6550 5550 6250
-Wire Wire Line
-	5550 6850 5550 7700
+Wire Wire Line
+	5850 6850 5850 7700
 $Comp
 L PS_Test_Grid-rescue:MCP6001R-RESCUE-PS_Test_Grid U3
@@
 	10600 7700 10600 7250
 Wire Wire Line
-	8900 6250 8900 6700
-Connection ~ 8900 6250
+	8900 6000 8900 6700
+Connection ~ 8900 6000
 Wire Wire Line
 	8900 7000 8900 7150
@@
 	10250 7300 10350 7300
 Connection ~ 10350 7300
-Text Notes 8400 6200 0    60   ~ 0
+Text Notes 8350 5900 0    60   ~ 0
 V divider resistors appear in parallel to the input\n220K = 110K\nUsing 220K and 2.2uF cuts off at .66Hz
 $Comp
@@
 Connection ~ 8550 7700
 Connection ~ 6250 7700
-Wire Wire Line
-	5850 6850 5850 7700
-Connection ~ 5850 7700
-Wire Wire Line
-	5550 6250 5850 6250
-Wire Wire Line
-	5550 7700 5850 7700
 Connection ~ 10600 7700
 $Comp
@@
 	12850 7050 13000 7050
 Wire Wire Line
-	12850 6250 12850 7050
+	12850 6000 12850 6250
 Wire Wire Line
 	13000 2900 12950 2900
@@
 Text Label 12350 2800 0    60   ~ 0
 S_1
-Text Notes 6550 6000 0    60   ~ 0
+Text Notes 6500 5800 0    60   ~ 0
 630nm Peak Sensitivity
-Text Notes 5500 6200 0    60   ~ 0
+Text Notes 5500 5900 0    60   ~ 0
 630nm Dominant\nVLDS1235R LED
-Text Notes 6700 2050 0    60   ~ 0
+Text Notes 6750 1750 0    60   ~ 0
 540nm Peak Sensitivity\nNOA1212CUTAG\n
-Text Notes 5650 2050 0    60   ~ 0
+Text Notes 5650 1750 0    60   ~ 0
 AM2520ZGC09\nGreen LED
-Wire Wire Line
-	5400 3550 5700 3550
 Wire Wire Line
 	10650 2700 9900 2700
@@
 	8050 3550 8750 3550
 Wire Wire Line
-	7950 2100 9150 2100
+	7950 1850 9150 1850
 Wire Wire Line
 	7150 3550 7700 3550
@@
 	7300 6850 7300 6950
 Wire Wire Line
-	8000 6250 8900 6250
+	8000 6000 8900 6000
 Wire Wire Line
 	7300 7700 7550 7700
@@
 	6050 3550 6300 3550
 Wire Wire Line
-	5700 3550 6050 3550
-Wire Wire Line
 	11550 2800 11700 2800
 Wire Wire Line
@@
 	6250 7700 7300 7700
 Wire Wire Line
-	5850 7700 6250 7700
-Wire Wire Line
 	10600 7700 12000 7700
 Wire Wire Line
@@
 Wire Wire Line
 	12250 2800 13000 2800
-Wire Wire Line
-	12250 3550 12650 3550
-Wire Wire Line
-	12000 7700 12450 7700
 Wire Wire Line
 	12000 6950 13000 6950
@@
 L Device:D_ALT D3
 U 1 1 5BFF69DD
-P 12650 3200
-F 0 "D3" V 12500 3300 50  0000 C CNN
-F 1 "D_ALT" V 12750 3350 50  0000 C CNN
-F 2 "Solutions:NSR20F30NXT5G_DIODE" H 12650 3200 50  0001 C CNN
-F 3 "~" H 12650 3200 50  0001 C CNN
-	1    12650 3200
-	0    1    1    0
+P 12400 2100
+F 0 "D3" H 12250 2000 50  0000 C CNN
+F 1 "D_ALT" H 12500 2000 50  0000 C CNN
+F 2 "Solutions:RB751S40T5G_DIODE" H 12400 2100 50  0001 C CNN
+F 3 "~" H 12400 2100 50  0001 C CNN
+	1    12400 2100
+	1    0    0    -1
 $EndComp
 $Comp
 L Device:D_ALT D4
 U 1 1 5BFF6A6F
-P 12450 7300
-F 0 "D4" V 12300 7400 50  0000 C CNN
-F 1 "D_ALT" V 12550 7450 50  0000 C CNN
-F 2 "Solutions:NSR20F30NXT5G_DIODE" H 12450 7300 50  0001 C CNN
-F 3 "~" H 12450 7300 50  0001 C CNN
-	1    12450 7300
-	0    1    1    0
-$EndComp
-Wire Wire Line
-	9150 2100 10850 2100
-Wire Wire Line
-	6050 2100 6400 2100
-Wire Wire Line
-	6250 6250 6250 6450
-Wire Wire Line
-	10600 6250 12450 6250
-Wire Wire Line
-	8900 6250 10600 6250
-Connection ~ 10600 6250
-Wire Wire Line
-	10600 6250 10600 6650
-Connection ~ 5850 6250
-Wire Wire Line
-	5850 6250 6250 6250
-Connection ~ 8000 6250
-Wire Wire Line
-	6900 6250 8000 6250
-Connection ~ 6900 6250
-Connection ~ 6250 6250
-Wire Wire Line
-	6250 6250 6900 6250
-Connection ~ 6050 2100
-Connection ~ 5700 2100
-Wire Wire Line
-	5700 2100 6050 2100
-Text Notes 12600 7600 0    50   ~ 0
-NSR20F30NXT5G
-Text Notes 12650 3450 0    50   ~ 0
-NSR20F30NXT5G
+P 12300 6250
+F 0 "D4" H 12150 6150 50  0000 C CNN
+F 1 "D_ALT" H 12500 6150 50  0000 C CNN
+F 2 "Solutions:RB751S40T5G_DIODE" H 12300 6250 50  0001 C CNN
+F 3 "~" H 12300 6250 50  0001 C CNN
+	1    12300 6250
+	1    0    0    -1
+$EndComp
+Wire Wire Line
+	6250 6000 6250 6450
+Connection ~ 8000 6000
+Text Notes 12050 6150 0    50   ~ 0
+RB751S40T5G
+Text Notes 12100 2000 0    50   ~ 0
+RB751S40T5G
+Wire Wire Line
+	6050 1850 7950 1850
+Wire Wire Line
+	9150 1850 12950 1850
+Wire Wire Line
+	12250 3550 12950 3550
+Wire Wire Line
+	12550 2100 12950 2100
+Connection ~ 12950 2100
+Wire Wire Line
+	12950 2100 12950 1850
+Wire Wire Line
+	12250 2100 10850 2100
+Wire Wire Line
+	5600 2100 5600 2500
 Wire Wire Line
 	6400 2200 6400 2100
 Connection ~ 6400 2100
 Wire Wire Line
-	6400 2100 6700 2100
-Wire Wire Line
 	6700 2200 6700 2100
 Connection ~ 6700 2100
 Wire Wire Line
-	6700 2100 7150 2100
+	6700 2100 6400 2100
 Wire Wire Line
 	7150 2400 7150 2100
 Connection ~ 7150 2100
 Wire Wire Line
-	7150 2100 7950 2100
+	7150 2100 6700 2100
 Wire Wire Line
 	10850 2500 10850 2100
 Connection ~ 10850 2100
 Wire Wire Line
-	10850 2100 12650 2100
-Wire Wire Line
-	12650 3050 12650 2100
-Connection ~ 12650 2100
-Wire Wire Line
-	12650 2100 12950 2100
-Wire Wire Line
-	12650 3350 12650 3550
-Connection ~ 12650 3550
-Wire Wire Line
-	12650 3550 12950 3550
-Wire Wire Line
-	12450 7150 12450 6250
-Connection ~ 12450 6250
+	10850 2100 7150 2100
+Text Label 11800 2100 0    50   ~ 0
+DVDD
+Wire Wire Line
+	6250 6000 8000 6000
+Wire Wire Line
+	8900 6000 12850 6000
+Wire Wire Line
+	12000 7700 12850 7700
 Wire Wire Line
 	12450 6250 12850 6250
-Wire Wire Line
-	12450 7450 12450 7700
-Connection ~ 12450 7700
-Wire Wire Line
-	12450 7700 12850 7700
+Connection ~ 12850 6250
+Wire Wire Line
+	12850 6250 12850 7050
+Wire Wire Line
+	12150 6250 10600 6250
+Wire Wire Line
+	5850 6250 5850 6550
+Wire Wire Line
+	6900 6350 6900 6250
+Connection ~ 6900 6250
+Wire Wire Line
+	10600 6650 10600 6250
+Connection ~ 10600 6250
+Wire Wire Line
+	10600 6250 6900 6250
+Text Label 11450 6250 0    50   ~ 0
+DVPP
+Wire Wire Line
+	5600 2100 6400 2100
+Wire Wire Line
+	5600 3550 6050 3550
+Wire Wire Line
+	5850 6250 6900 6250
+Wire Wire Line
+	5850 7700 6250 7700
 $EndSCHEMATC
